File: hw/7_seg_led_tht_3mm/7_seg_led_tht_3mm.kicad_pcb (KiCad board)
At the start: 2 copper layers, 160 x 60 mm, 291 parts, among them J1 USB_C_Plug_USB2.0, J2 Conn_02x05_Odd_Even, Q1 2N7002K, Q10 2N7002K, Q11 2N7002K, Q12 2N7002K, Q13 2N7002K, Q14 2N7002K, Q15 2N7002K, Q16 2N7002K, Q17 2N7002K, Q18 2N7002K, Q19 2N7002K, Q2 2N7002K, Q20 2N7002K, Q21 2N7002K, Q22 2N7002K, Q23 2N7002K, Q24 2N7002K, Q25 2N7002K, Q26 2N7002K, Q27 2N7002K, Q28 2N7002K, Q29 2N7002K, Q3 2N7002K, Q30 2N7002K, Q31 2N7002K, Q32 2N7002K, Q33 2N7002K, Q4 2N7002K, Q5 2N7002K, Q6 2N7002K, Q7 2N7002K, Q8 2N7002K, Q9 2N7002K, SW1 SW_MEC_5E, SW2 SW_MEC_5E, SW3 SW_MEC_5E, U1 MIC5504-3.3YM5, U2 STM32G030K8Tx, U3 74HCT595, U4 74HCT595, U5 74HCT595, U6 74HCT595, Y1 32K768

Commit message: better animations and hw files
Parts:
- removed D18, D65, D66: LED, LED_THT:LED_D3.0mm
- removed J2: Conn_02x05_Odd_Even, Connector_PinHeader_1.27mm:PinHeader_2x05_P1.27mm_Vertical_SMD
- removed JP34: Jumper_2_Small_Open, Jumper:SolderJumper-2_P1.3mm_Open_RoundedPad1.0x1.5mm
- removed Q32: 2N7002K, Package_TO_SOT_SMD:SOT-23
- removed R100, R28, R99: R, Resistor_SMD:R_0805_2012Metric
- removed R98: 10K, Resistor_SMD:R_0603_1608Metric
- removed TP1, TP2, TP3, TP4, TP5, TP7: Test Point, TestPoint:TestPoint_Pad_D1.5mm
- added D1: D_Zener, Diode_SMD:D_SMB, B.Cu at (188.6, 87.8)
- added G***: LOGO, LOGO, F.Cu at (55.0, 26.0)
- added G***: LOGO, LOGO, F.Cu at (188.0, 99.8)
- added G***: LOGO, LOGO, B.Cu at (195.3, 46.2)
- added J3: PGM5526, Connector_PinSocket_2.54mm:PinSocket_1x02_P2.54mm_Vertical, B.Cu at (189.3, 38.7)
- added J4: PGM5526, Connector_PinSocket_2.54mm:PinSocket_1x02_P2.54mm_Vertical, B.Cu at (195.5, 38.7)
- added J5: Conn_01x05, Connector_PinHeader_2.54mm:PinHeader_1x05_P2.54mm_Vertical, F.Cu at (202.9, 86.0)
- added REF**: ESD-Logo_6.6x6mm_SilkScreen, Symbol:ESD-Logo_6.6x6mm_SilkScreen, B.Cu at (145.7, 89.1)
- added REF**: CE-Logo_8.5x6mm_SilkScreen, Symbol:CE-Logo_8.5x6mm_SilkScreen, B.Cu at (155.3, 89.0)
- Y1: footprint Crystal:Crystal_SMD_3215-2Pin_3.2x1.5mm -> Crystal:Crystal_C26-LF_D2.1mm_L6.5mm_Vertical
- moved C9 73.9 mm to (193.9, 80.3), turned to -90 degrees
- moved C7 69.6 mm to (199.3, 77.3), turned to 0 degrees
- moved C6 69.6 mm to (199.3, 75.3), turned to 0 degrees
- moved C8 49.7 mm to (195.7, 80.3), turned to -90 degrees
- moved Y1 46.4 mm to (195.9, 75.4)
- moved U2 45.9 mm to (187.7, 79.7)
- moved C4 44.3 mm to (199.4, 81.3)
- moved R4 44.2 mm to (190.5, 43.0), turned to 180 degrees
- moved H1 42.4 mm to (48.0, 40.0)
- moved JP17 41.9 mm to (134.8, 69.0)
- moved Q15 41.9 mm to (131.5, 69.0)
- moved R47 41.9 mm to (128.8, 69.0)
- moved R48 41.9 mm to (137.1, 69.0)
- moved R49 41.9 mm to (139.1, 69.0)
- moved JP33 41.9 mm to (62.7, 69.1)
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Connections:
- Y1 pad 1: Net-(U2-PC15) -> Net-(U2-PC14)
- Y1 pad 2: Net-(U2-PC14) -> Net-(U2-PC15)
Routing:
- net VDD: track 0.00 -> 71.3 mm, vias 0 -> 1
- net Net-(Q33-D): track 0.00 -> 63.7 mm
- net +5V: track 102.7 -> 47.5 mm, vias 4 -> 7
- net /TEMP_analog: track 0.00 -> 52.5 mm, vias 0 -> 2
- net /LOGO_PWM: track 0.00 -> 49.7 mm, vias 0 -> 2
- net GND: track 97.6 -> 145.7 mm, vias 47 -> 63
- net /FD_analog: track 0.00 -> 47.4 mm, vias 0 -> 2
- net /SW_CLK: track 0.00 -> 33.7 mm, vias 0 -> 1
- net /SW_DIO: track 0.00 -> 33.3 mm, vias 0 -> 1
- net /7_SEG_2/QH: track 12.4 -> 39.2 mm
- net /7_SEG_3/QH: track 13.9 -> 39.9 mm
- net /SW_1: track 0.00 -> 23.7 mm
- net /7_SEG_4/QH: track 18.9 -> 0.00 mm, vias 2 -> 0
- net / T_{NRST}: track 0.00 -> 18.7 mm, vias 0 -> 2
- net Net-(D33-K): track 0.00 -> 16.5 mm
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- added copper zone on B.Cu, net +5V
Other:
- outline, holes or cut-outs redrawn
- board text added: "${TITLE} ${REVISION} ${ISSUE_DATE}"
- board text added: "1"
- board text added: "4"
- board text added: "5V 1A"
- board text added: "D2"
- board text added: "D3"
- board text added: "D5"
- board text added: "D6"
- board text added: "D7"
- board text added: "G2"
- board text added: "G3"
- board text added: "G5"
- board text added: "G6"
- board text added: "G7"
- board text added: "Made in Poland"
- board text added: "SET"
- board text added: "TGWLC 1.0"
